File: mss-crossover.kicad_sch (KiCad schematic)
At the start: 15 parts, among them J1 2x-screw, J2 RJ45, J4 2x-screw, J7 RJ45, Q1 2N3904

Commit message: Changed MPN for the RJ45 to RJHSE-5080
Parts:
- J2, J7: MPN MTJ-881X1 -> RJHSE-5080
Changed lines of the file:
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@@
       (effects (font (size 1.27 1.27)) hide)
     )
-    (property "Datasheet" "https://app.adam-tech.com/products/download/data_sheet/203793/mtj-881x1-data-sheet.pdf" (at 106.68 76.835 90)
+    (property "Datasheet" "" (at 106.68 76.835 90)
       (effects (font (size 1.27 1.27)) hide)
     )
@@
       (effects (font (size 1.27 1.27)))
     )
-    (property "MPN" "MTJ-881X1" (at 106.68 76.2 0)
+    (property "MPN" "RJHSE-5080" (at 106.68 76.2 0)
       (effects (font (size 1.27 1.27)) hide)
     )
@@
       (effects (font (size 1.27 1.27)) hide)
     )
-    (property "Datasheet" "https://app.adam-tech.com/products/download/data_sheet/203793/mtj-881x1-data-sheet.pdf" (at 177.8 76.835 90)
+    (property "Datasheet" "" (at 177.8 76.835 90)
       (effects (font (size 1.27 1.27)) hide)
     )
@@
       (effects (font (size 1.27 1.27)))
     )
-    (property "MPN" "MTJ-881X1" (at 177.8 76.2 0)
+    (property "MPN" "RJHSE-5080" (at 177.8 76.2 0)
       (effects (font (size 1.27 1.27)) hide)
     )

Commit message: Changed connectors to MJ3221-88 (the yellow ones that Ryan found) and put the connectors on opposite edges of the board (like everyone but me likes).  Also updated the footprint for the pulse transformer to have larger holes and to include the unused center pin.
Parts:
- J2, J7: footprint Imports:CONN_RJSBE5080_16P13X12P57_AMP -> myMods:MJ3221-88; MPN RJHSE-5080 -> MJ3221-88
- L1: footprint myMods:FIS101NL -> myMods:Murata_56300C
